Commit message: Actualización del material (2026-10-22)

File: mini_bot/urdf/mini_bot.urdf.xacro (robot description, xacro)
@@ -4,5 +4,6 @@
   Los nombres de links y joints ya están puestos: no los cambies, porque los launch,
   el bridge y los controladores de los ejercicios siguientes dependen de ellos.
-  Rellena lo que está marcado con TODO.
+  En el ejercicio 1, activa los PASOS comentados; en los siguientes, añade lo que pide
+  cada enunciado en su sección.
   Soluciones por ejercicio en  mini_bot/solutions/exNN/mini_bot.urdf.xacro
 -->
@@ -32,7 +33,9 @@
   <material name="dark"><color rgba="0.10 0.10 0.12 1.0"/></material>
   <!-- ============================ EJERCICIO 1: GEOMETRÍA ====================== -->
-  <!-- base_footprint: link vacío a ras de suelo. Es el frame que usarás en RViz. -->
+  <!-- La geometría ya está escrita, pero comentada. Actívala en tres pasos: en cada PASO, borra
+       las líneas marcadas con "(borra esta línea)" y relanza display.launch.py. -->
+  <!-- base_footprint: link vacío a ras de suelo. Es el frame fijo de RViz. -->
   <link name="${prefix}base_footprint"/>
-  <!-- base_link: ejemplo resuelto. Fíjate en el patrón visual + collision + inertial. -->
+  <!-- base_link: la caja. Patrón de todo link: visual + collision + inertial. -->
   <link name="${prefix}base_link">
     <visual>
@@ -50,19 +53,25 @@
     <parent link="${prefix}base_footprint"/>
     <child  link="${prefix}base_link"/>
-    <!-- TODO (1a): eleva la base hasta el eje de las ruedas.
-         Pista: wheel_r + base_z/2 - 0.02 -->
-    <origin xyz="0 0 0" rpy="0 0 0"/>
+    <!-- PASO 1: con este origen, la caja queda a medias bajo el suelo. El de debajo la eleva
+         hasta el eje de las ruedas. -->
+    <origin xyz="0 0 0" rpy="0 0 0"/> <!-- PASO 1 (borra esta línea) -->
+    <!-- PASO 1 (borra esta línea)
+    <origin xyz="0 0 ${wheel_r + base_z/2 - 0.02}" rpy="0 0 0"/>
+    fin del PASO 1 (borra esta línea) -->
   </joint>
-  <!-- Una sola macro para las dos ruedas. 'reflect' vale 1 (izquierda) o -1 (derecha). -->
+  <!-- PASO 2: las ruedas. Una macro, instanciada dos veces: 'reflect' vale 1 (izquierda)
+       o -1 (derecha) y pone cada rueda a un lado con el mismo código. -->
+  <!-- PASO 2 (borra esta línea)
   <xacro:macro name="wheel" params="side reflect">
     <link name="${prefix}${side}_wheel_link">
       <visual>
-        <!-- TODO (1b): cilindro de radio wheel_r y largo wheel_l.
-             Ojo con la orientación: el cilindro nace en Z, la rueda gira en Y → rpy="${pi/2} 0 0" -->
-        <origin xyz="0 0 0" rpy="0 0 0"/>
-        <geometry><box size="0.01 0.01 0.01"/></geometry>
+        <origin xyz="0 0 0" rpy="${pi/2} 0 0"/>
+        <geometry><cylinder radius="${wheel_r}" length="${wheel_l}"/></geometry>
         <material name="dark"/>
       </visual>
-      <!-- TODO (1c): la colisión, igual que el visual -->
+      <collision>
+        <origin xyz="0 0 0" rpy="${pi/2} 0 0"/>
+        <geometry><cylinder radius="${wheel_r}" length="${wheel_l}"/></geometry>
+      </collision>
       <xacro:cylinder_inertia m="${wheel_mass}" r="${wheel_r}" l="${wheel_l}"/>
     </link>
@@ -70,17 +79,38 @@
       <parent link="${prefix}base_link"/>
       <child  link="${prefix}${side}_wheel_link"/>
-      <!-- TODO (1d): coloca la rueda a media separación en Y, usando 'reflect',
-           y un poco por debajo del centro de la base -->
-      <origin xyz="0 0 0" rpy="0 0 0"/>
-      <!-- TODO (1e): eje de giro -->
-      <axis xyz="0 0 1"/>
+      <origin xyz="0 ${reflect * wheel_sep/2} ${-base_z/2 + 0.02}" rpy="0 0 0"/>
+      <axis xyz="0 1 0"/>
       <dynamics damping="0.05" friction="0.01"/>
     </joint>
+    <gazebo reference="${prefix}${side}_wheel_link">
+      <mu1>1.0</mu1>
+      <mu2>1.0</mu2>
+    </gazebo>
   </xacro:macro>
-  <!-- TODO (1f): instancia las dos ruedas con la macro de arriba.
-       <xacro:wheel side="left"  reflect="1"/> ... -->
-  <!-- TODO (1g): rueda loca delantera. Esfera de radio caster_r, joint fijo,
-       y en Gazebo rozamiento 0 para que no arrastre:
-         <gazebo reference="${prefix}caster_link"><mu1>0.0</mu1><mu2>0.0</mu2></gazebo> -->
+  <xacro:wheel side="left"  reflect="1"/>
+  <xacro:wheel side="right" reflect="-1"/>
+  fin del PASO 2 (borra esta línea) -->
+  <!-- PASO 3: la rueda loca. Una esfera con joint fijo y rozamiento 0 en Gazebo. -->
+  <!-- PASO 3 (borra esta línea)
+  <link name="${prefix}caster_link">
+    <visual>
+      <geometry><sphere radius="${caster_r}"/></geometry>
+      <material name="dark"/>
+    </visual>
+    <collision>
+      <geometry><sphere radius="${caster_r}"/></geometry>
+    </collision>
+    <xacro:sphere_inertia m="0.2" r="${caster_r}"/>
+  </link>
+  <joint name="caster_joint" type="fixed">
+    <parent link="${prefix}base_link"/>
+    <child  link="${prefix}caster_link"/>
+    <origin xyz="${base_x/2 - 0.05} 0 ${-base_z/2 - caster_r + 0.03}" rpy="0 0 0"/>
+  </joint>
+  <gazebo reference="${prefix}caster_link">
+    <mu1>0.0</mu1>
+    <mu2>0.0</mu2>
+  </gazebo>
+  fin del PASO 3 (borra esta línea) -->
   <!-- ============================ EJERCICIO 3: SENSORES ======================= -->
   <!-- Aquí irán lidar_link, camera_link y sus etiquetas <gazebo> con los sensores. -->

Commit message: Actualización del material (2026-10-23)

File: mini_bot/urdf/mini_bot.urdf.xacro (robot description, xacro)
@@ -4,7 +4,8 @@
   Los nombres de links y joints ya están puestos: no los cambies, porque los launch,
   el bridge y los controladores de los ejercicios siguientes dependen de ellos.
-  En el ejercicio 1, activa los PASOS comentados; en los siguientes, añade lo que pide
-  cada enunciado en su sección.
-  Soluciones por ejercicio en  mini_bot/solutions/exNN/mini_bot.urdf.xacro
+  Casi todo está escrito y comentado por PASOS. Los preámbulos dicen cuándo activar cada uno:
+  borra las líneas marcadas con "(borra esta línea)". En los ejercicios, pega lo que pida el
+  enunciado en su sección.
+  Soluciones en  mini_bot/solutions/preambulo_N/ y mini_bot/solutions/ejercicio_N/
 -->
 <robot xmlns:xacro="http://www.ros.org/wiki/xacro" name="mini_bot">
@@ -32,7 +33,6 @@
   <material name="accent_red"><color rgba="0.78 0.21 0.18 1.0"/></material>
   <material name="dark"><color rgba="0.10 0.10 0.12 1.0"/></material>
-  <!-- ============================ EJERCICIO 1: GEOMETRÍA ====================== -->
-  <!-- La geometría ya está escrita, pero comentada. Actívala en tres pasos: en cada PASO, borra
-       las líneas marcadas con "(borra esta línea)" y relanza display.launch.py. -->
+  <!-- ====================== PREÁMBULO 1: GEOMETRÍA ============================ -->
+  <!-- PASOS 1 a 3. Después de cada uno, relanza display.launch.py. -->
   <!-- base_footprint: link vacío a ras de suelo. Es el frame fijo de RViz. -->
   <link name="${prefix}base_footprint"/>
@@ -113,7 +113,127 @@
   </gazebo>
   fin del PASO 3 (borra esta línea) -->
-  <!-- ============================ EJERCICIO 3: SENSORES ======================= -->
-  <!-- Aquí irán lidar_link, camera_link y sus etiquetas <gazebo> con los sensores. -->
-  <!-- =========================== EJERCICIO 5: ros2_control ==================== -->
-  <!-- Aquí irán el bloque <ros2_control> y el plugin gz_ros2_control. -->
+  <!-- ====================== PREÁMBULO 2: SENSORES ============================= -->
+  <!-- Un link y un joint fijo para cada sensor, y una etiqueta <gazebo> con el <sensor>, que es lo
+       que Gazebo simula. ROS 2 ignora la etiqueta <gazebo>. Resoluciones y frecuencias bajas a
+       propósito: así la simulación sigue fluida sin GPU.
+       <topic>        dónde publica Gazebo: ${tns}/scan es /scan sin namespace y /robot_a/scan con él
+       <gz_frame_id>  el frame que llevarán los mensajes: sin él, Gazebo pondría su propio nombre -->
+  <!-- PASO 7: LiDAR, 180 muestras a 5 Hz entre -90° y +90°, de 0,12 a 8 m. Publica en Gazebo en ${tns}/scan. -->
+  <!-- PASO 7 (borra esta línea)
+  <link name="${prefix}lidar_link">
+    <visual>
+      <geometry><cylinder radius="0.035" length="0.04"/></geometry>
+      <material name="accent_red"/>
+    </visual>
+    <collision>
+      <geometry><cylinder radius="0.035" length="0.04"/></geometry>
+    </collision>
+    <xacro:cylinder_inertia m="0.15" r="0.035" l="0.04"/>
+  </link>
+  <joint name="lidar_joint" type="fixed">
+    <parent link="${prefix}base_link"/>
+    <child  link="${prefix}lidar_link"/>
+    <origin xyz="0.10 0 ${base_z/2 + 0.02}" rpy="0 0 0"/>
+  </joint>
+  <gazebo reference="${prefix}lidar_link">
+    <sensor name="lidar" type="gpu_lidar">
+      <topic>${tns}/scan</topic>
+      <gz_frame_id>${prefix}lidar_link</gz_frame_id>
+      <update_rate>5</update_rate>
+      <always_on>true</always_on>
+      <visualize>true</visualize>
+      <lidar>
+        <scan>
+          <horizontal>
+            <samples>180</samples>
+            <resolution>1</resolution>
+            <min_angle>-1.5708</min_angle>
+            <max_angle>1.5708</max_angle>
+          </horizontal>
+        </scan>
+        <range>
+          <min>0.12</min>
+          <max>8.0</max>
+          <resolution>0.02</resolution>
+        </range>
+      </lidar>
+    </sensor>
+  </gazebo>
+  fin del PASO 7 (borra esta línea) -->
+  <!-- PASO 8: cámara de 320 × 240 a 10 Hz, en el morro. Publica en Gazebo en ${tns}/camera/image. -->
+  <!-- PASO 8 (borra esta línea)
+  <link name="${prefix}camera_link">
+    <visual>
+      <geometry><box size="0.02 0.06 0.03"/></geometry>
+      <material name="accent_red"/>
+    </visual>
+    <xacro:box_inertia m="0.05" x="0.02" y="0.06" z="0.03"/>
+  </link>
+  <joint name="camera_joint" type="fixed">
+    <parent link="${prefix}base_link"/>
+    <child  link="${prefix}camera_link"/>
+    <origin xyz="${base_x/2 - 0.01} 0 ${base_z/2 - 0.01}" rpy="0 0 0"/>
+  </joint>
+  <gazebo reference="${prefix}camera_link">
+    <sensor name="camera" type="camera">
+      <topic>${tns}/camera/image</topic>
+      <gz_frame_id>${prefix}camera_link</gz_frame_id>
+      <update_rate>10</update_rate>
+      <always_on>true</always_on>
+      <camera>
+        <horizontal_fov>1.047</horizontal_fov>
+        <image>
+          <width>320</width>
+          <height>240</height>
+          <format>R8G8B8</format>
+        </image>
+        <clip>
+          <near>0.1</near>
+          <far>15.0</far>
+        </clip>
+      </camera>
+    </sensor>
+  </gazebo>
+  fin del PASO 8 (borra esta línea) -->
+  <!-- ====================== EJERCICIO 2: SENSORES NUEVOS ====================== -->
+  <!-- Pega aquí los sensores del ejercicio 2. -->
+  <!-- ====================== PREÁMBULO 3: ros2_control ========================= -->
+  <!-- PASO 11: el control. Dos piezas:
+       - <ros2_control>: qué joints se controlan y cómo. Cada rueda acepta órdenes de velocidad
+         (command_interface) y devuelve su posición y su velocidad (state_interface). El
+         <plugin> dice quién es el hardware: aquí, Gazebo.
+       - el plugin gz_ros2_control de Gazebo: arranca, dentro de la simulación, el
+         controller_manager de ROS 2, con los controladores declarados en controllers.yaml.
+       Los joints van sin ${prefix}: viven dentro del namespace del robot. -->
+  <!-- PASO 11 (borra esta línea)
+  <ros2_control name="${prefix}GazeboSimSystem" type="system">
+    <hardware>
+      <plugin>gz_ros2_control/GazeboSimSystem</plugin>
+    </hardware>
+    <joint name="left_wheel_joint">
+      <command_interface name="velocity">
+        <param name="min">-10.0</param>
+        <param name="max">10.0</param>
+      </command_interface>
+      <state_interface name="position"/>
+      <state_interface name="velocity"/>
+    </joint>
+    <joint name="right_wheel_joint">
+      <command_interface name="velocity">
+        <param name="min">-10.0</param>
+        <param name="max">10.0</param>
+      </command_interface>
+      <state_interface name="position"/>
+      <state_interface name="velocity"/>
+    </joint>
+  </ros2_control>
+  <gazebo>
+    <plugin filename="gz_ros2_control-system" name="gz_ros2_control::GazeboSimROS2ControlPlugin">
+      <parameters>$(find mini_bot)/config/controllers.yaml</parameters>
+      <ros>
+        <namespace>${ns}</namespace>
+      </ros>
+    </plugin>
+  </gazebo>
+  fin del PASO 11 (borra esta línea) -->
 </robot>
