Commit message: Actualización del material (2026-10-23)

File: mini_bot/solutions/ejercicio_2/mini_bot.urdf.xacro (robot description, xacro)
@@ -44,4 +44,11 @@
       <material name="body_grey"/>
     </visual>
+    <!-- La franja roja del morro: solo visual (sin collision), para saber hacia dónde mira el
+         robot. Un link puede tener tantos <visual> como haga falta. -->
+    <visual>
+      <origin xyz="${base_x/2 - 0.03} 0 ${base_z/2 + 0.0025}" rpy="0 0 0"/>
+      <geometry><box size="0.06 ${base_y} 0.005"/></geometry>
+      <material name="accent_red"/>
+    </visual>
     <collision>
       <origin xyz="0 0 0" rpy="0 0 0"/>

File: mini_bot/solutions/ejercicio_3/mast_bot.urdf.xacro (robot description, xacro)
@@ -41,4 +41,11 @@
       <material name="body_grey"/>
     </visual>
+    <!-- La franja roja del morro: solo visual (sin collision), para saber hacia dónde mira el
+         robot. Un link puede tener tantos <visual> como haga falta. -->
+    <visual>
+      <origin xyz="${base_x/2 - 0.03} 0 ${base_z/2 + 0.0025}" rpy="0 0 0"/>
+      <geometry><box size="0.06 ${base_y} 0.005"/></geometry>
+      <material name="accent_red"/>
+    </visual>
     <collision>
       <origin xyz="0 0 0" rpy="0 0 0"/>

File: mini_bot/solutions/preambulo_1/mini_bot.urdf.xacro (robot description, xacro)
@@ -44,4 +44,11 @@
       <material name="body_grey"/>
     </visual>
+    <!-- La franja roja del morro: solo visual (sin collision), para saber hacia dónde mira el
+         robot. Un link puede tener tantos <visual> como haga falta. -->
+    <visual>
+      <origin xyz="${base_x/2 - 0.03} 0 ${base_z/2 + 0.0025}" rpy="0 0 0"/>
+      <geometry><box size="0.06 ${base_y} 0.005"/></geometry>
+      <material name="accent_red"/>
+    </visual>
     <collision>
       <origin xyz="0 0 0" rpy="0 0 0"/>

File: mini_bot/solutions/preambulo_2/mini_bot.urdf.xacro (robot description, xacro)
@@ -44,4 +44,11 @@
       <material name="body_grey"/>
     </visual>
+    <!-- La franja roja del morro: solo visual (sin collision), para saber hacia dónde mira el
+         robot. Un link puede tener tantos <visual> como haga falta. -->
+    <visual>
+      <origin xyz="${base_x/2 - 0.03} 0 ${base_z/2 + 0.0025}" rpy="0 0 0"/>
+      <geometry><box size="0.06 ${base_y} 0.005"/></geometry>
+      <material name="accent_red"/>
+    </visual>
     <collision>
       <origin xyz="0 0 0" rpy="0 0 0"/>

File: mini_bot/solutions/preambulo_3/mini_bot.urdf.xacro (robot description, xacro)
@@ -44,4 +44,11 @@
       <material name="body_grey"/>
     </visual>
+    <!-- La franja roja del morro: solo visual (sin collision), para saber hacia dónde mira el
+         robot. Un link puede tener tantos <visual> como haga falta. -->
+    <visual>
+      <origin xyz="${base_x/2 - 0.03} 0 ${base_z/2 + 0.0025}" rpy="0 0 0"/>
+      <geometry><box size="0.06 ${base_y} 0.005"/></geometry>
+      <material name="accent_red"/>
+    </visual>
     <collision>
       <origin xyz="0 0 0" rpy="0 0 0"/>

File: mini_bot/urdf/mast_bot.urdf.xacro (robot description, xacro)
@@ -41,4 +41,11 @@
       <material name="body_grey"/>
     </visual>
+    <!-- La franja roja del morro: solo visual (sin collision), para saber hacia dónde mira el
+         robot. Un link puede tener tantos <visual> como haga falta. -->
+    <visual>
+      <origin xyz="${base_x/2 - 0.03} 0 ${base_z/2 + 0.0025}" rpy="0 0 0"/>
+      <geometry><box size="0.06 ${base_y} 0.005"/></geometry>
+      <material name="accent_red"/>
+    </visual>
     <collision>
       <origin xyz="0 0 0" rpy="0 0 0"/>

File: mini_bot/urdf/mini_bot.urdf.xacro (robot description, xacro)
@@ -44,4 +44,11 @@
       <material name="body_grey"/>
     </visual>
+    <!-- La franja roja del morro: solo visual (sin collision), para saber hacia dónde mira el
+         robot. Un link puede tener tantos <visual> como haga falta. -->
+    <visual>
+      <origin xyz="${base_x/2 - 0.03} 0 ${base_z/2 + 0.0025}" rpy="0 0 0"/>
+      <geometry><box size="0.06 ${base_y} 0.005"/></geometry>
+      <material name="accent_red"/>
+    </visual>
     <collision>
       <origin xyz="0 0 0" rpy="0 0 0"/>

Commit message: Actualización del material (2026-10-26)

File: mini_bot/solutions/ejercicio_2/mini_bot.urdf.xacro (robot description, xacro)
@@ -228,6 +228,6 @@
   </gazebo>
   <!-- "Ultrasonido": Gazebo no tiene sensor de ultrasonidos, así que se imita con un lidar de
-       5 rayos en un cono de 15° y 3 m de alcance, a 10 Hz. Va inclinado 0,1 rad hacia arriba:
-       el robot cabecea 0,067 rad hacia delante en reposo y, recto, el sensor vería el suelo a 1 m. -->
+       5 rayos en un cono de 15° y 3 m de alcance, a 10 Hz. Va detrás, mirando hacia atrás (giro
+       de 180° en el joint): delante ya mira el LiDAR, y así sus medidas no se mezclan. -->
   <link name="${prefix}ultrasound_link">
     <visual>
@@ -241,5 +241,5 @@
     <parent link="${prefix}base_link"/>
     <child  link="${prefix}ultrasound_link"/>
-    <origin xyz="${base_x/2 + 0.005} 0 0" rpy="0 -0.1 0"/>
+    <origin xyz="${-base_x/2 - 0.005} 0 0" rpy="0 0 ${pi}"/>
   </joint>
   <gazebo reference="${prefix}ultrasound_link">

Commit message: Actualización del material (2026-10-26)

File: mini_bot/solutions/ejercicio_2/mini_bot.urdf.xacro (robot description, xacro)
@@ -229,5 +229,7 @@
   <!-- "Ultrasonido": Gazebo no tiene sensor de ultrasonidos, así que se imita con un lidar de
        5 rayos en un cono de 15° y 3 m de alcance, a 10 Hz. Va detrás, mirando hacia atrás (giro
-       de 180° en el joint): delante ya mira el LiDAR, y así sus medidas no se mezclan. -->
+       de 180° en el joint): delante ya mira el LiDAR, y así sus medidas no se mezclan. Y va
+       inclinado 0,067 rad hacia abajo: el robot cabecea hacia delante en reposo, así que la parte
+       de atrás queda levantada; con la inclinación, el rayo sale horizontal. -->
   <link name="${prefix}ultrasound_link">
     <visual>
@@ -241,5 +243,5 @@
     <parent link="${prefix}base_link"/>
     <child  link="${prefix}ultrasound_link"/>
-    <origin xyz="${-base_x/2 - 0.005} 0 0" rpy="0 0 ${pi}"/>
+    <origin xyz="${-base_x/2 - 0.005} 0 0" rpy="0 0.067 ${pi}"/>
   </joint>
   <gazebo reference="${prefix}ultrasound_link">
